File: FL-Ver0.7.brd (EAGLE design)
At the start: 77 x 30 mm, 29 parts, among them Q1 SS8050SMDSMD, Q2 IRF540, Q3 8550, Q4 8050, Q5 SS8050SMDSMD

Commit message: 2013-09-30
設計印製板
Parts:
- removed LED1, LED2, LED3: (no value), led:LED5MM
- removed MOSI, RST, SCK: (no value), _wirepad:1,6/0,8
- removed PAD3, PAD4, PAD5: (no value), _wirepad:SMD2,54-5,08
- removed Q2: IRF540, transistor-fet:TO220
- removed Q3: 8550, _mylbr:SOT23-BEC
- removed Q4: 8050, _mylbr:SOT23-BEC
- removed Q5: SS8050SMDSMD, _mylbr:SOT23-BEC
- removed R4: 5k1, _myrc:M0805
- removed R7: (no value), _myrc:M0805
- added +, -: (no value), _wirepad:1,6/0,9
- added IN: (no value), _con-molex:22-23-2031
- added OUT, SUPPLY: (no value), _con-molex:22-23-2021
- added Q10: IRF540, transistor-fet:TO220
- added Q6, Q7, Q8, Q9: (no value), _mylbr:SOT23-BEC
- added R0: (no value), _resistor:P0613/15
- added R10: 10, _myrc:M0805
- C3: device inductor-rcl-2:153CLV-0605 -> _resistor:153CLV-0807
- Q1: value SS8050SMDSMD -> 8050
- R1: device _myrc:M1206 -> _myrc:M0805
- R2: value (none) -> 10k
- R5: value 10 -> (none)
- R6: value (none) -> 5k1
- R8: value 10k -> (none)
- moved C3 132.3 mm to (70.5, 23.5)
- moved R3 104.9 mm to (11.6, 15.2), turned to 180 degrees
- moved D1 103.9 mm to (60.3, 23.5), turned to 180 degrees
- moved L1 86.5 mm to (47.6, 22.9), turned to 180 degrees
- moved R1 85.0 mm to (11.4, 22.9), turned to 180 degrees
- moved C2 66.7 mm to (30.5, 15.9), turned to 180 degrees
- moved R5 48.1 mm to (17.1, 22.9), turned to 180 degrees
- moved Q1 38.8 mm to (10.8, 10.2), turned to 90 degrees
- moved R8 33.3 mm to (17.1, 15.2)
- moved R2 15.2 mm to (11.4, 19.1), turned to 0 degrees
- moved R6 10.9 mm to (17.1, 19.1), turned to 0 degrees
- moved C1 7.01 mm to (26.0, 5.71)
- moved U$1 6.02 mm to (18.4, 6.99)
- moved JP1 1.42 mm to (5.71, 5.08)
Connections:
- removed net N$14: LED1.K, LED2.A
- removed net N$15: LED2.K, LED3.A
- removed net N$5: D1.A, L1.1, Q2.2
- new net FET-D: D1.A, L1.1, Q10.2
- new net N$1: Q6.C, Q9.B, R6.1
- new net N$17: Q7.C, R8.1
- net +5V: now also IN.1, Q8.E, R2.1, R3.2, SUPPLY.1; no longer PAD3.1, Q5.C, R4.2, R8.1
- net GND: now also IN.2, Q10.3, Q6.E, Q7.E, Q9.E, R0.1, SUPPLY.2; no longer PAD4.1, Q2.3, Q3.C, Q4.E, R1.1
- net N$10: now also IN.3, R1.2; no longer PAD5.1, R7.2
- net N$11: now also +.1, OUT.1; no longer LED1.A
- net N$12: now also JP1.4, R5.2; no longer MOSI.1, R2.2
- net N$13: now also Q1.C, R2.2; no longer Q4.C, R8.2
- net N$16: now also -.1, OUT.2, R0.2; no longer LED3.K, R1.2
- net N$2: now also JP1.3; no longer SCK.1
- net N$3: now also Q6.B, Q7.B, R5.1; no longer Q1.B, R2.1
- net N$4: now also JP1.5, R3.1; no longer R6.1, RST.1
- net N$6: now also Q8.B, R8.2; no longer Q1.C, Q3.B, Q5.B, R4.1
- net N$7: now also Q8.C, R10.1; no longer Q2.1, R5.1
- net N$8: now also Q10.1, Q9.C, R10.2; no longer Q3.E, Q5.E, R5.2
- net N$9: now also Q1.B, R1.1; no longer Q4.B, R7.1
Routing:
- net +5V: track 0.00 -> 96.7 mm
- net N$16: track 0.00 -> 62.5 mm
- net N$4: track 0.00 -> 47.4 mm, vias 0 -> 1
- net GND: track 0.00 -> 39.7 mm, vias 0 -> 5
- net FET-D: track 0.00 -> 35.9 mm
- net N$11: track 0.00 -> 33.9 mm
- net N$12: track 0.00 -> 30.0 mm, vias 0 -> 2
- net N$8: track 0.00 -> 24.8 mm
- net N$1: track 0.00 -> 23.3 mm
- net N$13: track 0.00 -> 22.5 mm, vias 0 -> 2
- net N$9: track 0.00 -> 18.0 mm, vias 0 -> 2
- net N$6: track 0.00 -> 17.4 mm, vias 0 -> 2
- net N$3: track 0.00 -> 17.2 mm, vias 0 -> 2
- net N$10: track 0.00 -> 15.6 mm, vias 0 -> 1
- net N$17: track 0.00 -> 14.9 mm, vias 0 -> 2
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- added copper zone on layer 1, net FET-D
- added copper zone on layer 16, net GND
