File: FL-Ver0.7.sch (EAGLE design)
At the start: 29 parts, among them Q1 SS8050SMDSMD, Q2 IRF540, Q3 8550, Q4 8050, Q5 SS8050SMDSMD

Commit message: 2013-09-30
設計印製板
Parts:
- removed LED1, LED2, LED3: (no value), led:LED5MM
- removed MOSI, RST, SCK: (no value), _wirepad:1,6/0,8
- removed PAD3, PAD4, PAD5: (no value), _wirepad:SMD5
- removed Q3: 8550, _mylbr:SS8550SMDSMD
- removed Q4: 8050, _mylbr:SS8050SMDSMD
- removed Q5: SS8050SMDSMD, _mylbr:SS8050SMDSMD
- removed R4: 5k1, _myrc:R-EU_M0805
- removed R7: (no value), _myrc:R-EU_M0805
- added +, -: (no value), _wirepad:1,6/0,9
- added IN: 22-23-2031, _con-molex:22-23-2031
- added OUT, SUPPLY: 22-23-2021, _con-molex:22-23-2021
- added Q6, Q7, Q9: SS8050SMDSMD, _mylbr:SS8050SMDSMD
- added Q8: SS8550SMDSMD, _mylbr:SS8550SMDSMD
- added R0: (no value), _resistor:R-EU_0613/15
- added R10: 10, _myrc:R-EU_M0805
- C3: device inductor-rcl-2:CPOL-EU153CLV-0605 -> _resistor:CPOL-EU153CLV-0807
- Q1: value SS8050SMDSMD -> 8050
- R1: device _myrc:R-EU_M1206 -> _myrc:R-EU_M0805
- R2: value (none) -> 10k
- R5: value 10 -> (none)
- R6: value (none) -> 5k1
- R8: value 10k -> (none)
- renumbered Q2 to Q10
Connections:
- net N$5 renamed FET-D
- removed net N$14: LED1.C, LED2.A
- removed net N$15: LED2.C, LED3.A
- new net N$1: Q6.C, Q9.B, R6.1
- new net N$17: Q7.C, R8.1
- net +5V: now also IN-1.S, Q8.E, R2.1, R3.2, SUPPLY-1.S; no longer PAD3.P, Q5.C, R4.2, R8.1
- net GND: now also IN-2.S, Q6.E, Q7.E, Q9.E, R0.1, SUPPLY-2.S; no longer PAD4.P, Q3.C, Q4.E, R1.1
- net N$10: now also IN-3.S, R1.2; no longer PAD5.P, R7.2
- net N$11: now also +.P, OUT-1.S; no longer LED1.A
- net N$12: now also JP1.4, R5.2; no longer MOSI.P, R2.2
- net N$13: now also Q1.C, R2.2; no longer Q4.C, R8.2
- net N$16: now also -.P, OUT-2.S, R0.2; no longer LED3.C, R1.2
- net N$2: now also JP1.3; no longer SCK.P
- net N$3: now also Q6.B, Q7.B, R5.1; no longer Q1.B, R2.1
- net N$4: now also JP1.5, R3.1; no longer R6.1, RST.P
- net N$6: now also Q8.B, R8.2; no longer Q1.C, Q3.B, Q5.B, R4.1
- net N$7: now also Q8.C, R10.1; no longer Q10.G, R5.1
- net N$8: now also Q10.G, Q9.C, R10.2; no longer Q3.E, Q5.E, R5.2
- net N$9: now also Q1.B, R1.1; no longer Q4.B, R7.1
Other:
- moved on the sheet: C2, JP1, Q1, R1, R2, R3, R5, R6, R8
